File: variador.sch (KiCad schematic (older format))
At the start: 81 parts, among them CON1 BDM, CON2 CONN_3, CON3 CONN_4, CON4 CONN_3, CON5 CONN_3, CON6 CONN_2, Q1 TRIAC, Q2 TRIAC, Q3 TRIAC, T1 TRANSFO, T2 TRANSFO, U1 MC9S08SH8, U2 LM339, U3 OPTO-TRIAC, U4 OPTO-TRIAC, U5 OPTO-TRIAC, U6 7805, X1 12 MHZ

Commit message: backup
Parts:
- removed C3, C7: 25 pF, symbol C
- removed CON2: CONN_3, symbol CONN_3
- removed D7: LED, symbol LED
- removed X1: 12 MHZ, symbol CRYSTAL
- added C23: C, symbol C-RESCUE-variador
- added C24: 1 uF, symbol CAPAPOL
- added C3: C0.1 uF, symbol C-RESCUE-variador
- added CON2: CONN_2, symbol CONN_2
- added D1: LED_RABG, symbol LED_RABG
- added R34: 10K, symbol R-RESCUE-variador
- added RV1: POT, symbol POT
- C1, C10, C12, C13, C14, C15, C16, C17, C18, C19, C2, C20, C21, C22, C5, C6, C8, C9: symbol C -> C-RESCUE-variador
- D6: symbol LED -> LED-RESCUE-variador
- R1, R10, R11, R12, R13, R14, R15, R16, R17, R18, R19, R2, R20, R21, R22, R23, R24, R25, R28, R29, R3, R30, R31, R32, R33, R4, R5, R7, R8, R9: symbol R -> R-RESCUE-variador
- U2: symbol LM339 -> LM339-RESCUE-variador
- U3, U4, U5: symbol OPTO-TRIAC -> OPTO-TRIAC-RESCUE-variador
Connections:
- net GND: now also R21.2, C23.2, C3.2, CON2.2 (PM); no longer R21.1
- net vreg: now also C23.1, C24.1, R34.2
- net EXTAL renamed B
- net B: now also D1.1 (RED_CATHODE)
- net Led1 renamed R
- net R: now also D1.3 (BLUE_CATHODE)
- net RxD: no longer names the net of U1.16 (PTB0/PIB0/RxD/ADP4)
- net RxD: now also C3.1, RV1.2
- net TxD renamed PM
- net PM: now also JP1.1, R24.2, C24.2
- net XTAL renamed G
- net G: now also D1.4 (GREEN_CATHODE)
- removed net c_Flash: JP1.1, R24.2, U1.17 (PTA3/PIA3/SCL/ADP3)
- new net: D1.2 (COMMON_ANODE), R21.1
- new net NM: CON2.1 (P1), R34.1, U1.17 (PTA3/PIA3/SCL/ADP3)
- no-connect marks 8 -> 9
Other:
- moved on the sheet: C16, CON3, CON4, CON5, CON6, JP1, R21, R23
