File: pot.sch (KiCad schematic (older format))
At the start: 103 parts, among them CON1 JP, CON2 SELECT, CON3 BDM, CON4 SENSOR, IC1 4N25, P1 CONN_2, P2 CONN_1, P3 CONN_1, P4 CONN_1, P5 CONN_1, P6 CONN_1, P7 CONN_1, P8 CONN_1, Q1 BC548, Q2 TRIAC, Q3 TRIAC, Q4 TRIAC, T1 TRANSFO, U1 LM339, U2 MC9S08SH8, U3 7805, U4 OPTO-TRIAC, U5 OPTO-TRIAC, U6 OPTO-TRIAC, X1 12 MHZ

Commit message: ultimo commit febrero
Parts:
- C1, C11, C12, C13, C14, C15, C16, C17, C18, C19, C2, C20, C3, C4, C6, C7, C8, C9: symbol C -> C-RESCUE-pot
- D2, D4: symbol LED -> LED-RESCUE-pot
- IC1: symbol 4N25 -> 4N25-RESCUE-pot
- POT1: symbol POT -> POT-RESCUE-pot
- R1, R10, R11, R12, R13, R14, R15, R16, R17, R18, R19, R2, R20, R21, R22, R23, R24, R25, R26, R27, R28, R29, R3, R30, R31, R32, R4, R5, R6, R7, R8, R9: symbol R -> R-RESCUE-pot
- RL1: symbol RM50-XX11 -> RM50-xx11
- U1: symbol LM339 -> LM339-RESCUE-pot
- U4, U5, U6: symbol OPTO-TRIAC -> OPTO-TRIAC-RESCUE-pot
Other:
- moved on the sheet: C1, C10, C11, C12, C13, C14, C15, C16, C17, C18, C19, C2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
